File: mu-ltz.sch (KiCad schematic (older format))
At the start: 47 parts, among them J10 TRIM2, J2 GND, J3 Hi, J5 Lo, J6 Vin+, J9 TRIM1, Q1 MMBT3904LT1G, U1 LTZ1000, U2 AD8667, U3 ADA4523-1

Commit message: Rev. 0.2 layout finished, not yet tested
Parts:
- removed C13: 100nF, Capacitor_SMD:C_0603_1608Metric, symbol Device:C
- removed FB2: Ferrite_Bead_Small, Inductor_SMD:L_0603_1608Metric, symbol Device:Ferrite_Bead_Small
- removed Q1: MMBT3904LT1G, Package_TO_SOT_SMD:SOT-23, symbol Device:Q_NPN_BEC
- added JP3: Jumper_NO_Small, Jumper:SolderJumper-2_P1.3mm_Open_RoundedPad1.0x1.5mm, symbol Device:Jumper_NO_Small
- added Q1: 2SD1628G-TD-E, Package_TO_SOT_SMD:SOT-89-3, symbol Device:Q_NPN_BCE
- R6: value 400k -> dnp
- RN1: value 13k 1k -> 13k1k
- renumbered J2 to J1, J5 to J2, J3 to J4, JP3 to JP4, JP4 to JP5
Connections:
- net GND: now also D1.1 (K), J1.1 (Pin_1), J2.1 (Pin_1), JP1.1, R18.1, R4.1, RN1.1, U1.7 (TS+TC_E)
- net VCC: now also R8.2, Q1.2 (C)
- net at C2.2, R6.1, U1.1 (Heater+): now also Q1.3 (E)
- net at U1.3 (Zener+): now also D2.1 (K), R1.1, R10.2, R2.1, RN1.3; no longer R10.1
- net at R3.2: now also Q1.1 (B)
- net at J10.1 (Pin_1), JP1.2, JP2.1: now also JP3.1; no longer JP4.2
- net at C17.1, JP4.1, JP5.1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: no longer R14.2
- new net: R10.1, U3.3 (+)
- new net: JP3.2, JP4.2, R14.2
Other:
- moved on the sheet: C1, C2, C3, C5, D2, J10, J9, JP1, JP2, JP4, JP5, R1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
